File: reloj.sch (KiCad schematic (older format))
At the start: 83 parts, among them J1 Conn_01x03, J2 USB_B_Mini, SW1 SW_Push, SW2 SW_Push, U1 LM555, U10 74LS90, U11 74LS92, U12 74LS90, U13 74LS08, U14 74LS90, U15 74LS47, U16 74LS47, U17 74LS47, U18 74LS47, U19 SA04-11SRWA, U2 74LS90, U20 SA04-11SRWA, U21 SA04-11SRWA, U22 SA04-11SRWA, U3 74LS90, U4 74LS90, U5 74LS90, U6 CD4060B, U7 74LS90, U8 74LS90, U9 74LS92, Y1 32768Hz

Commit message: Change LED resistors to 1k to dim them a bit
Change 555 timer R1 to 330ohm to reduce BOM complexity
Parts:
- R1: value 220 -> 330; DKPN CF18JT220RCT-ND‎ -> CF18JT330RCT-ND‎; MPN ‎CF18JT220R‎ -> ‎CF18JT330R‎
- R10, R11, R12, R13, R14, R15, R16, R17, R18, R19, R20, R21, R22, R23, R24, R25, R26, R27, R28, R29, R30, R31, R32, R33, R34, R35, R8, R9: value 330 -> 1k; DKPN CF18JT330RCT-ND‎ -> CF18JT1K00CT-DN; MPN ‎CF18JT330R‎ -> ‎CF18JT1K00
